File: tiny20/chopped choc/tiny20C.kicad_pcb (KiCad board)
At the start: 2 copper layers, 94.3 x 60 mm, 14 parts

Commit message: added gerbers for the chopped version
Parts:
- moved S1 222.9 mm to (182.7, 148.6)
- moved S3 222.9 mm to (200.9, 132.1)
- moved S5 222.9 mm to (218.9, 127.0)
- moved B1 222.9 mm to (187.6, 121.0)
- moved B2 222.9 mm to (187.6, 121.0)
- moved S10 222.9 mm to (255.9, 158.1)
- moved S4 222.9 mm to (200.9, 121.0)
- moved S6 222.9 mm to (218.9, 116.0)
- moved S7 222.9 mm to (236.9, 133.1)
- moved S8 222.9 mm to (236.9, 122.0)
- moved S9 222.9 mm to (244.9, 158.1)
- moved MCU1 222.9 mm to (254.9, 131.6)
- moved S2 222.9 mm to (181.7, 137.6)
- moved REF** 220.8 mm to (181.0, 114.4)
Connections:
- REF** pad 3: P8 -> P7
- S1 pad 1: P1 -> P10
- S2 pad 1: P2 -> P16
- S3 pad 1: P3 -> P14
- S4 pad 1: P4 -> P19
- S5 pad 1: P5 -> P15
- S6 pad 1: P6 -> P20
- S7 pad 1: P7 -> P18
- S8 pad 1: P8 -> P21
- S9 pad 1: P10 -> P8
Routing:
- net P7: track 0.00 -> 96.9 mm
- net VCC: track 0.00 -> 91.9 mm
- net RST: track 0.00 -> 85.4 mm, vias 0 -> 2
- net P10: track 0.00 -> 76.8 mm
- net P16: track 0.00 -> 75.3 mm
- net P19: track 0.00 -> 57.9 mm
- net P14: track 0.00 -> 54.1 mm
- net P20: track 0.00 -> 44.0 mm
- net P15: track 0.00 -> 40.0 mm
- net P8: track 0.00 -> 36.9 mm
- net P21: track 0.00 -> 21.7 mm
- net P9: track 0.00 -> 18.7 mm
- net P18: track 0.00 -> 16.0 mm
- added copper zone on B.Cu, net GND
- added copper zone on F.Cu, net GND
Other:
- board size 94.3 x 60 mm -> 93.9 x 60.2 mm
- net class Default removed
