File: tiny20/chopped thumbs/tiny20TC.kicad_pcb (KiCad board)
At the start: 2 copper layers, 94.8 x 61 mm, 14 parts

Commit message: added gerbers for the chopped version
Parts:
- moved B1 216.7 mm to (168.0, 125.7)
- moved B2 216.7 mm to (168.0, 125.7)
- moved S1 214.2 mm to (162.4, 156.6)
- moved S2 214.2 mm to (160.9, 139.6)
- moved S4 214.2 mm to (180.6, 123.0)
- moved S5 214.2 mm to (198.6, 135.0)
- moved S3 214.2 mm to (180.6, 140.0)
- moved MCU1 214.2 mm to (234.6, 133.5)
- moved S10 214.2 mm to (235.6, 161.0)
- moved S6 214.2 mm to (198.6, 118.0)
- moved S7 214.2 mm to (216.6, 141.0)
- moved S8 214.2 mm to (216.6, 124.0)
- moved S9 214.2 mm to (224.6, 161.0)
- moved REF** 212.2 mm to (159.4, 117.5)
Routing:
- added copper zone on B.Cu, net GND
- added copper zone on F.Cu, net GND
Other:
- net class Default removed
