File: tiny20/choc/tiny20.kicad_pcb (KiCad board)
At the start: 2 copper layers, 94.8 x 61 mm, 14 parts

Commit message: updated the pcb
Regular choc spacing board is finished with a new edgecut and promicro compatibility
Parts:
- removed the REF** at (16.6, -39.5)
- added BT01: Battery_Cell, keyboard-footprints:battery_pads_reversible, B.Cu at (280.3, 137.0)
- added REF**: TRRS-PJ-320A-dual, keyboard-footprints:TRS, F.Cu at (202.5, 104.6)
- added SW01: SW_SPDT, keyboard-footprints:Power_reversible, F.Cu at (276.3, 103.7)
- B1: footprint E73:SW_TACT_ALPS_SKQGABE010 -> keyboard-footprints:SW_TACT_ALPS_SKQGABE010
- B2: footprint E73:SW_TACT_ALPS_SKQGABE010 -> keyboard-footprints:SW_TACT_ALPS_SKQGABE010; moved to B.Cu
- MCU1: footprint ProMicro -> keyboard-footprints:ProMicro_minimal
- S1, S10, S2, S3, S4, S5, S6, S7, S8, S9: footprint PG1350 -> keyboard-footprints:chocV1_reversible
- moved B1 236.8 mm to (208.6, 111.8)
- moved B2 236.8 mm to (208.6, 111.8), turned to -90 degrees
- moved S1 235.2 mm to (203.8, 142.5)
- moved S6 235.2 mm to (240.0, 104.0)
- moved S9 235.2 mm to (260.0, 147.0)
- moved S8 235.2 mm to (258.0, 110.0)
- moved S3 235.2 mm to (222.0, 126.0)
- moved S4 235.2 mm to (222.0, 109.0)
- moved MCU1 235.2 mm to (276.1, 119.5)
- moved S2 235.2 mm to (202.3, 125.6)
- moved S10 235.2 mm to (277.0, 147.0)
- moved S5 235.2 mm to (240.0, 121.0)
- moved S7 235.2 mm to (258.0, 127.0)
Connections:
- S1 pad 1: P1 -> GND
- S1 pad 2: GND -> P21
- S10 pad 1: P9 -> GND
- S10 pad 2: GND -> P9
- S2 pad 1: P2 -> GND
- S2 pad 2: GND -> P20
- S3 pad 1: P3 -> GND
- S3 pad 2: GND -> P19
- S4 pad 1: P4 -> GND
- S4 pad 2: GND -> P18
- S5 pad 1: P5 -> GND
- S5 pad 2: GND -> P15
- S6 pad 1: P6 -> GND
- S6 pad 2: GND -> P14
- S7 pad 1: P7 -> GND
- S7 pad 2: GND -> P16
- S8 pad 1: P8 -> GND
- S8 pad 2: GND -> P10
- S9 pad 1: P10 -> GND
- S9 pad 2: GND -> P8
Routing:
- net VCC: track 0.00 -> 152.8 mm
- net P1: track 0.00 -> 147.5 mm
- net RST: track 0.00 -> 142.6 mm, vias 0 -> 2
- net P20: track 0.00 -> 103.6 mm
- net P18: track 0.00 -> 94.4 mm
- net P21: track 0.00 -> 93.6 mm
- net P19: track 0.00 -> 81.1 mm
- net P14: track 0.00 -> 73.5 mm
- net P15: track 0.00 -> 59.5 mm
- net P10: track 0.00 -> 39.6 mm
- net pm: track 0.00 -> 38.0 mm, vias 0 -> 2
- net P16: track 0.00 -> 29.5 mm
- net P8: track 0.00 -> 24.6 mm
- net P9: track 0.00 -> 21.0 mm
- net RAW: track 0.00 -> 19.1 mm
- added copper zone on B.Cu, net GND
- added copper zone on F.Cu, net GND
Other:
- board size 94.8 x 61 mm -> 93.7 x 62.2 mm
- net class Default removed
